Commit message: Kienmatics Updatae in Simand Keyboard teleop

File: 30_ros2_ws/src/guardian_description/urdf/guardian_sim.urdf.xacro (robot description, xacro)
@@ -1,4 +1,4 @@
 <?xml version="1.0"?>
-<robot name="guardian" xmlns:xacro="http://www.ros.org/wiki/xacro">
+<robot name="guardian" xmlns:xacro="http://www.ros.org/wiki/xacro" xmlns:gz="http://gazebosim.org/schema">
   <!-- ── Materials ─────────────────────────────────────────────────────────── -->
   <material name="dark_grey"><color rgba="0.2 0.2 0.2 1.0"/></material>
@@ -26,6 +26,13 @@
   </link>
   <!-- ── Wheels ────────────────────────────────────────────────────────────── -->
-  <!-- Wheel axles at z=0.0748 (wheel_radius) so wheels rest on z=0 ground    -->
-  <xacro:macro name="wheel" params="name x y">
+  <!-- Wheel axles at z=0.0748 (wheel_radius) so wheels rest on z=0 ground.
+       fdir1 gives each wheel anisotropic friction (mu along the roller's
+       rolling direction, mu2~=0 across it) approximating real mecanum
+       rollers — without this the wheels behave like plain isotropic-grip
+       round wheels, which fights MecanumDrive's commanded wheel velocities
+       and produces oscillating (forward/backward/forward) motion instead
+       of a clean strafe. Opposite corners share roller orientation (FL+RR,
+       FR+RL), matching the physical X-roller-pattern of a mecanum wheel set. -->
+  <xacro:macro name="wheel" params="name x y roller_dir">
     <link name="${name}_wheel">
       <visual>
@@ -54,13 +61,22 @@
     </joint>
     <gazebo reference="${name}_wheel">
-      <mu1>1.0</mu1>
-      <mu2>1.0</mu2>
       <material>Gazebo/Blue</material>
+      <collision>
+        <surface>
+          <friction>
+            <ode>
+              <mu>1.0</mu>
+              <mu2>0.0</mu2>
+              <fdir1 gz:expressed_in="base_link">${roller_dir}</fdir1>
+            </ode>
+          </friction>
+        </surface>
+      </collision>
     </gazebo>
   </xacro:macro>
-  <xacro:wheel name="front_left"  x=" 0.0856" y=" 0.120"/>
-  <xacro:wheel name="front_right" x=" 0.0856" y="-0.120"/>
-  <xacro:wheel name="rear_left"   x="-0.0856" y=" 0.120"/>
-  <xacro:wheel name="rear_right"  x="-0.0856" y="-0.120"/>
+  <xacro:wheel name="front_left"  x=" 0.0856" y=" 0.120" roller_dir="1 -1 0"/>
+  <xacro:wheel name="front_right" x=" 0.0856" y="-0.120" roller_dir="1 1 0"/>
+  <xacro:wheel name="rear_left"   x="-0.0856" y=" 0.120" roller_dir="1 1 0"/>
+  <xacro:wheel name="rear_right"  x="-0.0856" y="-0.120" roller_dir="1 -1 0"/>
   <!-- ── Lidar link ────────────────────────────────────────────────────────── -->
   <link name="laser">
@@ -121,14 +137,21 @@
     </sensor>
   </gazebo>
-  <!-- ── Gazebo: DiffDrive plugin ──────────────────────────────────────────── -->
-  <!-- Groups FL+BL as left, FR+BR as right — approximates mecanum for SLAM   -->
+  <!-- ── Gazebo: MecanumDrive plugin ───────────────────────────────────────── -->
+  <!-- True holonomic drive — DiffDrive (previously here) silently ignores
+       linear.y and cannot strafe at all, which defeated the entire point of
+       DWB's holonomic config (min_vel_y/max_vel_y) and this rover's mecanum
+       wheels. wheelbase/wheel_separation taken from the actual wheel joint
+       origins below (x=+-0.0856, y=+-0.120), not robot_params.yaml's
+       wheel_base_length (0.25) which is for the real robot's serial_bridge_node
+       and doesn't match this URDF's geometry. -->
   <gazebo>
-    <plugin filename="gz-sim-diff-drive-system"
-            name="gz::sim::systems::DiffDrive">
-      <left_joint>front_left_wheel_joint</left_joint>
-      <left_joint>rear_left_wheel_joint</left_joint>
-      <right_joint>front_right_wheel_joint</right_joint>
-      <right_joint>rear_right_wheel_joint</right_joint>
+    <plugin filename="gz-sim-mecanum-drive-system"
+            name="gz::sim::systems::MecanumDrive">
+      <front_left_joint>front_left_wheel_joint</front_left_joint>
+      <front_right_joint>front_right_wheel_joint</front_right_joint>
+      <back_left_joint>rear_left_wheel_joint</back_left_joint>
+      <back_right_joint>rear_right_wheel_joint</back_right_joint>
       <wheel_separation>0.240</wheel_separation>
+      <wheelbase>0.1712</wheelbase>
       <wheel_radius>0.0748</wheel_radius>
       <odom_publish_frequency>50</odom_publish_frequency>

Commit message: cad to ursf skript plus impelmtsaion in sim

File: 30_ros2_ws/src/guardian_description/urdf/guardian_sim.urdf.xacro (robot description, xacro)
@@ -1,4 +1,11 @@
 <?xml version="1.0"?>
 <robot name="guardian" xmlns:xacro="http://www.ros.org/wiki/xacro" xmlns:gz="http://gazebosim.org/schema">
+  <!-- Measured wheel_base_length/width/radius and lidar mount offsets —
+       AUTO-GENERATED from the CAD assembly by
+       20_hardware/cad/step_to_description.py. When a new CAD revision
+       replaces the current one, re-run that script (it overwrites
+       dimensions.xacro and meshes/*.stl); nothing below should ever need
+       hand-editing to track a CAD update. -->
+  <xacro:include filename="$(find guardian_description)/urdf/dimensions.xacro"/>
   <!-- ── Materials ─────────────────────────────────────────────────────────── -->
   <material name="dark_grey"><color rgba="0.2 0.2 0.2 1.0"/></material>
@@ -6,14 +13,19 @@
   <material name="red">     <color rgba="0.8 0.1 0.1 1.0"/></material>
   <!-- ── Chassis ───────────────────────────────────────────────────────────── -->
-  <!-- base_link origin at ground level; chassis box centred at z=0.05 (half height) -->
+  <!-- base_link origin at ground level, centred under the wheel footprint
+       (matches the origin step_to_description.py re-centers the CAD on).
+       Visual uses the real CAD mesh; collision stays a simple box sized
+       off the measured footprint — a full-detail collision mesh is a
+       common cause of jittery/unstable physics in Gazebo, so the real
+       geometry is visual-only. -->
   <link name="base_link">
     <visual>
-      <origin xyz="0 0 0.05" rpy="0 0 0"/>
-      <geometry><box size="0.2312 0.200 0.100"/></geometry>
+      <origin xyz="0 0 0" rpy="0 0 0"/>
+      <geometry><mesh filename="package://guardian_description/meshes/chassis.stl"/></geometry>
       <material name="dark_grey"/>
     </visual>
     <collision>
-      <origin xyz="0 0 0.05" rpy="0 0 0"/>
-      <geometry><box size="0.2312 0.200 0.100"/></geometry>
+      <origin xyz="0 0 ${wheel_radius}" rpy="0 0 0"/>
+      <geometry><box size="${wheel_base_length + 2*wheel_radius} ${wheel_base_width} ${2*wheel_radius}"/></geometry>
     </collision>
     <inertial>
@@ -36,12 +48,18 @@
   <xacro:macro name="wheel" params="name x y roller_dir">
     <link name="${name}_wheel">
+      <!-- No rpy on the visual: step_to_description.py already exports
+           wheel.stl with the disc face normal to Y (matching the joint's
+           `axis xyz="0 1 0"` below) — the 90deg X rotation below is only
+           needed for the collision <cylinder>, which URDF always models
+           Z-aligned by default. Applying it to the visual too was double
+           -rotating the mesh off its true spin axis. -->
       <visual>
-        <origin xyz="0 0 0" rpy="1.5708 0 0"/>
-        <geometry><cylinder radius="0.0748" length="0.05"/></geometry>
+        <origin xyz="0 0 0" rpy="0 0 0"/>
+        <geometry><mesh filename="package://guardian_description/meshes/wheel.stl"/></geometry>
         <material name="blue"/>
       </visual>
       <collision>
         <origin xyz="0 0 0" rpy="1.5708 0 0"/>
-        <geometry><cylinder radius="0.0748" length="0.05"/></geometry>
+        <geometry><cylinder radius="${wheel_radius}" length="0.05"/></geometry>
       </collision>
       <inertial>
@@ -56,5 +74,5 @@
       <parent link="base_link"/>
       <child  link="${name}_wheel"/>
-      <origin xyz="${x} ${y} 0.0748" rpy="0 0 0"/>
+      <origin xyz="${x} ${y} ${wheel_radius}" rpy="0 0 0"/>
       <axis xyz="0 1 0"/>
       <dynamics damping="0.01"/>
@@ -75,65 +93,85 @@
     </gazebo>
   </xacro:macro>
-  <xacro:wheel name="front_left"  x=" 0.0856" y=" 0.120" roller_dir="1 -1 0"/>
-  <xacro:wheel name="front_right" x=" 0.0856" y="-0.120" roller_dir="1 1 0"/>
-  <xacro:wheel name="rear_left"   x="-0.0856" y=" 0.120" roller_dir="1 1 0"/>
-  <xacro:wheel name="rear_right"  x="-0.0856" y="-0.120" roller_dir="1 -1 0"/>
-  <!-- ── Lidar link ────────────────────────────────────────────────────────── -->
-  <link name="laser">
-    <visual>
-      <origin xyz="0 0 0.015" rpy="0 0 0"/>
-      <geometry><cylinder radius="0.04" length="0.03"/></geometry>
-      <material name="red"/>
-    </visual>
-    <collision>
-      <origin xyz="0 0 0.015" rpy="0 0 0"/>
-      <geometry><cylinder radius="0.04" length="0.03"/></geometry>
-    </collision>
-    <inertial>
-      <mass value="0.1"/>
-      <inertia ixx="0.0001" ixy="0" ixz="0"
-               iyy="0.0001" iyz="0"
-               izz="0.0001"/>
-    </inertial>
-  </link>
-  <joint name="laser_joint" type="fixed">
-    <parent link="base_link"/>
-    <child  link="laser"/>
-    <origin xyz="0.0 0.0 0.175" rpy="0 0 0"/>
-  </joint>
+  <!-- x/y taken from wheel_base_length/width (measured off the CAD by
+       step_to_description.py), not hand-typed — regenerating
+       dimensions.xacro from a new CAD revision updates these for free. -->
+  <xacro:wheel name="front_left"  x="${ wheel_base_length/2}" y="${ wheel_base_width/2}" roller_dir="1 -1 0"/>
+  <xacro:wheel name="front_right" x="${ wheel_base_length/2}" y="${-wheel_base_width/2}" roller_dir="1 1 0"/>
+  <xacro:wheel name="rear_left"   x="${-wheel_base_length/2}" y="${ wheel_base_width/2}" roller_dir="1 1 0"/>
+  <xacro:wheel name="rear_right"  x="${-wheel_base_length/2}" y="${-wheel_base_width/2}" roller_dir="1 -1 0"/>
+  <!-- ── Lidar links ───────────────────────────────────────────────────────── -->
+  <!-- One reusable macro for both the front and back mount — the CAD has
+       an identical LIDAR unit at each end (lidar_front_*/lidar_back_* from
+       dimensions.xacro). gz_topic must differ per instance: Gazebo sensor
+       topics are per-link, and ros_gz_bridge's simple CLI form requires
+       the same name on the ROS and GZ sides (see the bridge arguments in
+       guardian.launch.py), so each gets its own raw topic before being
+       relayed through its own lidar_republisher_node. -->
+  <xacro:macro name="lidar" params="name x y z gz_topic yaw:=0">
+    <link name="${name}">
+      <visual>
+        <origin xyz="0 0 0" rpy="0 0 0"/>
+        <geometry><mesh filename="package://guardian_description/meshes/lidar.stl"/></geometry>
+        <material name="red"/>
+      </visual>
+      <collision>
+        <origin xyz="0 0 0.015" rpy="0 0 0"/>
+        <geometry><cylinder radius="0.04" length="0.03"/></geometry>
+      </collision>
+      <inertial>
+        <mass value="0.1"/>
+        <inertia ixx="0.0001" ixy="0" ixz="0"
+                 iyy="0.0001" iyz="0"
+                 izz="0.0001"/>
+      </inertial>
+    </link>
+    <!-- yaw: the front and back units are the same physical sensor mounted
+         at opposite ends, each rotated so its own "forward" (angle=0)
+         points outward away from the chassis — the back unit needs a
+         180deg yaw here, or its scan's angle=0 would point back into the
+         robot instead of away from it. This same yaw must be used by
+         lidar_merger_node when transforming each sensor's points into
+         base_link (see guardian.launch.py's front_yaw/back_yaw params). -->
+    <joint name="${name}_joint" type="fixed">
+      <parent link="base_link"/>
+      <child  link="${name}"/>
+      <origin xyz="${x} ${y} ${z}" rpy="0 0 ${yaw}"/>
+    </joint>
+    <gazebo reference="${name}">
+      <sensor name="gpu_lidar_${name}" type="gpu_lidar">
+        <pose>0 0 0.015 0 0 0</pose>
+        <topic>${gz_topic}</topic>
+        <gz_frame_id>${name}</gz_frame_id>
+        <update_rate>5</update_rate>
+        <lidar>
+          <scan>
+            <horizontal>
+              <samples>500</samples>
+              <resolution>1</resolution>
+              <min_angle>-3.14159265</min_angle>
+              <max_angle>3.14159265</max_angle>
+            </horizontal>
+          </scan>
+          <range>
+            <min>0.1</min>
+            <max>20.0</max>
+            <resolution>0.01</resolution>
+          </range>
+          <noise>
+            <type>gaussian</type>
+            <mean>0.0</mean>
+            <stddev>0.01</stddev>
+          </noise>
+        </lidar>
+        <always_on>true</always_on>
+        <visualize>true</visualize>
+      </sensor>
+    </gazebo>
+  </xacro:macro>
+  <xacro:lidar name="laser"      x="${lidar_front_x}" y="${lidar_front_y}" z="${lidar_front_z}" yaw="0"        gz_topic="/scan"/>
+  <xacro:lidar name="laser_back" x="${lidar_back_x}"  y="${lidar_back_y}"  z="${lidar_back_z}"  yaw="3.14159265" gz_topic="/scan_back"/>
   <!-- ── Gazebo: chassis colour ────────────────────────────────────────────── -->
   <gazebo reference="base_link">
     <material>Gazebo/DarkGrey</material>
-  </gazebo>
-  <!-- ── Gazebo: GPU Lidar sensor ──────────────────────────────────────────── -->
-  <gazebo reference="laser">
-    <sensor name="gpu_lidar" type="gpu_lidar">
-      <pose>0 0 0.015 0 0 0</pose>
-      <topic>/scan</topic>
-      <gz_frame_id>laser</gz_frame_id>
-      <update_rate>5</update_rate>
-      <lidar>
-        <scan>
-          <horizontal>
-            <samples>500</samples>
-            <resolution>1</resolution>
-            <min_angle>-3.14159265</min_angle>
-            <max_angle>3.14159265</max_angle>
-          </horizontal>
-        </scan>
-        <range>
-          <min>0.1</min>
-          <max>20.0</max>
-          <resolution>0.01</resolution>
-        </range>
-        <noise>
-          <type>gaussian</type>
-          <mean>0.0</mean>
-          <stddev>0.01</stddev>
-        </noise>
-      </lidar>
-      <always_on>true</always_on>
-      <visualize>true</visualize>
-    </sensor>
   </gazebo>
   <!-- ── Gazebo: MecanumDrive plugin ───────────────────────────────────────── -->
@@ -141,8 +179,8 @@
        linear.y and cannot strafe at all, which defeated the entire point of
        DWB's holonomic config (min_vel_y/max_vel_y) and this rover's mecanum
-       wheels. wheelbase/wheel_separation taken from the actual wheel joint
-       origins below (x=+-0.0856, y=+-0.120), not robot_params.yaml's
-       wheel_base_length (0.25) which is for the real robot's serial_bridge_node
-       and doesn't match this URDF's geometry. -->
+       wheels. wheel_separation/wheelbase/wheel_radius come from
+       dimensions.xacro (measured off the CAD), matching
+       mecanum_kinematics_node's wheel_base_length/width in robot_params.yaml
+       instead of an independently hand-typed placeholder. -->
   <gazebo>
     <plugin filename="gz-sim-mecanum-drive-system"
@@ -152,7 +190,7 @@
       <back_left_joint>rear_left_wheel_joint</back_left_joint>
       <back_right_joint>rear_right_wheel_joint</back_right_joint>
-      <wheel_separation>0.240</wheel_separation>
-      <wheelbase>0.1712</wheelbase>
-      <wheel_radius>0.0748</wheel_radius>
+      <wheel_separation>${wheel_base_width}</wheel_separation>
+      <wheelbase>${wheel_base_length}</wheelbase>
+      <wheel_radius>${wheel_radius}</wheel_radius>
       <odom_publish_frequency>50</odom_publish_frequency>
       <topic>/cmd_vel</topic>
