Commit message: Refactor robot description and launch configurations BIG CLEANUP

File: 30_ros2_ws/src/guardian_description/urdf/guardian.urdf.xacro (robot description, xacro)
@@ -1,34 +1,43 @@
 <?xml version="1.0"?>
-<robot name="guardian" xmlns:xacro="http://www.ros.org/wiki/xacro">
+<!-- Single robot description for both sim and real hardware. The <gazebo>
+     blocks below (MecanumDrive plugin, gpu_lidar sensors) are only ever
+     acted on by Gazebo — robot_state_publisher and RViz treat <gazebo> as
+     a standard, safely-ignorable URDF extension, so there's no need to
+     conditionally strip them out for real-hardware use. Previously this
+     was two near-duplicate files (guardian_sim.urdf.xacro +
+     guardian.urdf.xacro); the real-hardware copy silently never got any
+     of the CAD-mesh/dual-LIDAR updates made to the sim copy. -->
+<robot name="guardian" xmlns:xacro="http://www.ros.org/wiki/xacro" xmlns:gz="http://gazebosim.org/schema">
+  <!-- Measured wheel_base_length/width/radius and lidar mount offsets —
+       AUTO-GENERATED from the CAD assembly by
+       20_hardware/cad/step_to_description.py. When a new CAD revision
+       replaces the current one, re-run that script (it overwrites
+       dimensions.xacro and meshes/*.stl); nothing below should ever need
+       hand-editing to track a CAD update. -->
+  <xacro:include filename="$(find guardian_description)/urdf/dimensions.xacro"/>
   <!-- ── Materials ─────────────────────────────────────────────────────────── -->
-  <material name="dark_grey">
-    <color rgba="0.2 0.2 0.2 1.0"/>
-  </material>
-  <material name="blue">
-    <color rgba="0.1 0.4 0.8 1.0"/>
-  </material>
-  <material name="red">
-    <color rgba="0.8 0.1 0.1 1.0"/>
-  </material>
-  <!-- ── Chassis (base_link centre = ground level) ─────────────────────────── -->
-  <!--  Physical size: 231.2 mm × 200 mm × 100 mm                               -->
+  <material name="dark_grey"><color rgba="0.2 0.2 0.2 1.0"/></material>
+  <material name="blue">    <color rgba="0.1 0.4 0.8 1.0"/></material>
+  <material name="red">     <color rgba="0.8 0.1 0.1 1.0"/></material>
+  <!-- ── Chassis ───────────────────────────────────────────────────────────── -->
+  <!-- base_link origin at ground level, centred under the wheel footprint
+       (matches the origin step_to_description.py re-centers the CAD on).
+       Visual uses the real CAD mesh; collision stays a simple box sized
+       off the measured footprint — a full-detail collision mesh is a
+       common cause of jittery/unstable physics in Gazebo, so the real
+       geometry is visual-only. -->
   <link name="base_link">
     <visual>
-      <origin xyz="0 0 0.05" rpy="0 0 0"/>
-      <geometry>
-        <box size="0.2312 0.200 0.100"/>
-      </geometry>
+      <origin xyz="0 0 0" rpy="0 0 0"/>
+      <geometry><mesh filename="package://guardian_description/meshes/chassis.stl"/></geometry>
       <material name="dark_grey"/>
     </visual>
     <collision>
-      <origin xyz="0 0 0.05" rpy="0 0 0"/>
-      <geometry>
-        <box size="0.2312 0.200 0.100"/>
-      </geometry>
+      <origin xyz="0 0 ${wheel_radius}" rpy="0 0 0"/>
+      <geometry><box size="${wheel_base_length + 2*wheel_radius} ${wheel_base_width} ${2*wheel_radius}"/></geometry>
     </collision>
     <inertial>
       <origin xyz="0 0 0.05" rpy="0 0 0"/>
       <mass value="4.0"/>
-      <!-- box inertia: m/12*(h²+d²) etc. for 0.2312×0.200×0.100, m=4 kg -->
       <inertia ixx="0.01517" ixy="0" ixz="0"
                iyy="0.02250" iyz="0"
@@ -36,26 +45,37 @@
     </inertial>
   </link>
-  <!-- ── Wheels (continuous joints, visual only) ───────────────────────────── -->
-  <!-- wheel radius ~50 mm assumed; adjust if different -->
-  <xacro:macro name="wheel" params="name x y">
+  <!-- ── Wheels ────────────────────────────────────────────────────────────── -->
+  <!-- Wheel axles at z=wheel_radius so wheels rest on z=0 ground.
+       fdir1 (Gazebo-only, harmless elsewhere) gives each wheel anisotropic
+       friction (mu along the roller's rolling direction, mu2~=0 across it)
+       approximating real mecanum rollers — without this the wheels behave
+       like plain isotropic-grip round wheels, which fights MecanumDrive's
+       commanded wheel velocities and produces oscillating
+       (forward/backward/forward) motion instead of a clean strafe.
+       Opposite corners share roller orientation (FL+RR, FR+RL), matching
+       the physical X-roller-pattern of a mecanum wheel set. -->
+  <xacro:macro name="wheel" params="name x y roller_dir">
     <link name="${name}_wheel">
+      <!-- No rpy on the visual: step_to_description.py already exports
+           wheel.stl with the disc face normal to Y (matching the joint's
+           `axis xyz="0 1 0"` below) — the 90deg X rotation below is only
+           needed for the collision <cylinder>, which URDF always models
+           Z-aligned by default. Applying it to the visual too was double
+           -rotating the mesh off its true spin axis. -->
       <visual>
-        <origin xyz="0 0 0" rpy="1.5708 0 0"/>
-        <geometry>
-          <cylinder radius="0.05" length="0.04"/>
-        </geometry>
+        <origin xyz="0 0 0" rpy="0 0 0"/>
+        <geometry><mesh filename="package://guardian_description/meshes/wheel.stl"/></geometry>
         <material name="blue"/>
       </visual>
       <collision>
         <origin xyz="0 0 0" rpy="1.5708 0 0"/>
-        <geometry>
-          <cylinder radius="0.05" length="0.04"/>
-        </geometry>
+        <geometry><cylinder radius="${wheel_radius}" length="0.05"/></geometry>
       </collision>
       <inertial>
-        <mass value="0.3"/>
-        <inertia ixx="0.000375" ixy="0" ixz="0"
-                 iyy="0.000375" iyz="0"
-                 izz="0.000375"/>
+        <mass value="0.5"/>
+        <!-- solid cylinder: ixx=iyy=m(3r²+h²)/12, izz=mr²/2 -->
+        <inertia ixx="0.001561" ixy="0" ixz="0"
+                 iyy="0.001561" iyz="0"
+                 izz="0.001401"/>
       </inertial>
     </link>
@@ -63,41 +83,144 @@
       <parent link="base_link"/>
       <child  link="${name}_wheel"/>
-      <origin xyz="${x} ${y} 0" rpy="0 0 0"/>
+      <origin xyz="${x} ${y} ${wheel_radius}" rpy="0 0 0"/>
       <axis xyz="0 1 0"/>
+      <dynamics damping="0.01"/>
     </joint>
+    <gazebo reference="${name}_wheel">
+      <material>Gazebo/Blue</material>
+      <collision>
+        <surface>
+          <friction>
+            <ode>
+              <mu>1.0</mu>
+              <mu2>0.0</mu2>
+              <fdir1 gz:expressed_in="base_link">${roller_dir}</fdir1>
+            </ode>
+          </friction>
+        </surface>
+      </collision>
+    </gazebo>
   </xacro:macro>
-  <xacro:wheel name="front_left"  x=" 0.0856"  y=" 0.120"/>
-  <xacro:wheel name="front_right" x=" 0.0856"  y="-0.120"/>
-  <xacro:wheel name="rear_left"   x="-0.0856"  y=" 0.120"/>
-  <xacro:wheel name="rear_right"  x="-0.0856"  y="-0.120"/>
-  <!-- ── Scanse Sweep LIDAR ─────────────────────────────────────────────────── -->
-  <!--  Mounted middle-front at top surface:                                      -->
-  <!--    x = +0.1156 m (front half), y = 0 (centre), z = 0.100 m (top surface)  -->
-  <link name="laser">
-    <visual>
-      <origin xyz="0 0 0.015" rpy="0 0 0"/>
-      <geometry>
-        <cylinder radius="0.04" length="0.03"/>
-      </geometry>
-      <material name="red"/>
-    </visual>
-    <collision>
-      <origin xyz="0 0 0.015" rpy="0 0 0"/>
-      <geometry>
-        <cylinder radius="0.04" length="0.03"/>
-      </geometry>
-    </collision>
-    <inertial>
-      <mass value="0.1"/>
-      <inertia ixx="0.0001" ixy="0" ixz="0"
-               iyy="0.0001" iyz="0"
-               izz="0.0001"/>
-    </inertial>
-  </link>
-  <joint name="laser_joint" type="fixed">
-    <parent link="base_link"/>
-    <child  link="laser"/>
-    <!-- front edge centre, top surface of chassis -->
-    <origin xyz="0.1156 0.0 0.100" rpy="0 0 0"/>
-  </joint>
+  <!-- x/y taken from wheel_base_length/width (measured off the CAD by
+       step_to_description.py), not hand-typed — regenerating
+       dimensions.xacro from a new CAD revision updates these for free. -->
+  <xacro:wheel name="front_left"  x="${ wheel_base_length/2}" y="${ wheel_base_width/2}" roller_dir="1 -1 0"/>
+  <xacro:wheel name="front_right" x="${ wheel_base_length/2}" y="${-wheel_base_width/2}" roller_dir="1 1 0"/>
+  <xacro:wheel name="rear_left"   x="${-wheel_base_length/2}" y="${ wheel_base_width/2}" roller_dir="1 1 0"/>
+  <xacro:wheel name="rear_right"  x="${-wheel_base_length/2}" y="${-wheel_base_width/2}" roller_dir="1 -1 0"/>
+  <!-- ── Lidar links ───────────────────────────────────────────────────────── -->
+  <!-- One reusable macro for both the front and back mount — the CAD has
+       an identical LIDAR unit at each end (lidar_front_*/lidar_back_* from
+       dimensions.xacro). gz_topic (Gazebo-only) must differ per instance:
+       Gazebo sensor topics are per-link, and ros_gz_bridge's simple CLI
+       form requires the same name on the ROS and GZ sides (see the bridge
+       arguments in guardian.launch.py), so each gets its own raw topic
+       before being relayed through its own lidar_republisher_node. Real
+       hardware gets its scan data from l3xz_sweep_scanner_node instead —
+       these links only need to exist so robot_state_publisher can provide
+       the base_link -> laser/laser_back TF, which AMCL/Nav2/
+       lidar_merger_node all need regardless of sim or real. -->
+  <xacro:macro name="lidar" params="name x y z gz_topic yaw:=0">
+    <link name="${name}">
+      <visual>
+        <origin xyz="0 0 0" rpy="0 0 0"/>
+        <geometry><mesh filename="package://guardian_description/meshes/lidar.stl"/></geometry>
+        <material name="red"/>
+      </visual>
+      <collision>
+        <origin xyz="0 0 0.015" rpy="0 0 0"/>
+        <geometry><cylinder radius="0.04" length="0.03"/></geometry>
+      </collision>
+      <inertial>
+        <mass value="0.1"/>
+        <inertia ixx="0.0001" ixy="0" ixz="0"
+                 iyy="0.0001" iyz="0"
+                 izz="0.0001"/>
+      </inertial>
+    </link>
+    <!-- yaw: the front and back units are the same physical sensor mounted
+         at opposite ends, each rotated so its own "forward" (angle=0)
+         points outward away from the chassis — the back unit needs a
+         180deg yaw here, or its scan's angle=0 would point back into the
+         robot instead of away from it. This same yaw must be used by
+         lidar_merger_node when transforming each sensor's points into
+         base_link (see guardian.launch.py's front_yaw/back_yaw params). -->
+    <joint name="${name}_joint" type="fixed">
+      <parent link="base_link"/>
+      <child  link="${name}"/>
+      <origin xyz="${x} ${y} ${z}" rpy="0 0 ${yaw}"/>
+    </joint>
+    <gazebo reference="${name}">
+      <sensor name="gpu_lidar_${name}" type="gpu_lidar">
+        <pose>0 0 0.015 0 0 0</pose>
+        <topic>${gz_topic}</topic>
+        <gz_frame_id>${name}</gz_frame_id>
+        <update_rate>5</update_rate>
+        <lidar>
+          <scan>
+            <horizontal>
+              <samples>500</samples>
+              <resolution>1</resolution>
+              <min_angle>-3.14159265</min_angle>
+              <max_angle>3.14159265</max_angle>
+            </horizontal>
+          </scan>
+          <range>
+            <min>0.1</min>
+            <max>20.0</max>
+            <resolution>0.01</resolution>
+          </range>
+          <noise>
+            <type>gaussian</type>
+            <mean>0.0</mean>
+            <stddev>0.01</stddev>
+          </noise>
+        </lidar>
+        <always_on>true</always_on>
+        <visualize>true</visualize>
+      </sensor>
+    </gazebo>
+  </xacro:macro>
+  <xacro:lidar name="laser"      x="${lidar_front_x}" y="${lidar_front_y}" z="${lidar_front_z}" yaw="0"        gz_topic="/scan"/>
+  <xacro:lidar name="laser_back" x="${lidar_back_x}"  y="${lidar_back_y}"  z="${lidar_back_z}"  yaw="3.14159265" gz_topic="/scan_back"/>
+  <!-- ── Gazebo: chassis colour ────────────────────────────────────────────── -->
+  <gazebo reference="base_link">
+    <material>Gazebo/DarkGrey</material>
+  </gazebo>
+  <!-- ── Gazebo: MecanumDrive plugin ───────────────────────────────────────── -->
+  <!-- True holonomic drive — DiffDrive (previously here) silently ignores
+       linear.y and cannot strafe at all, which defeated the entire point of
+       DWB's holonomic config (min_vel_y/max_vel_y) and this rover's mecanum
+       wheels. wheel_separation/wheelbase/wheel_radius come from
+       dimensions.xacro (measured off the CAD), matching
+       mecanum_kinematics_node's wheel_base_length/width in robot_params.yaml
+       instead of an independently hand-typed placeholder. Only acted on by
+       Gazebo — harmless, unread content on real hardware. -->
+  <gazebo>
+    <plugin filename="gz-sim-mecanum-drive-system"
+            name="gz::sim::systems::MecanumDrive">
+      <front_left_joint>front_left_wheel_joint</front_left_joint>
+      <front_right_joint>front_right_wheel_joint</front_right_joint>
+      <back_left_joint>rear_left_wheel_joint</back_left_joint>
+      <back_right_joint>rear_right_wheel_joint</back_right_joint>
+      <wheel_separation>${wheel_base_width}</wheel_separation>
+      <wheelbase>${wheel_base_length}</wheelbase>
+      <wheel_radius>${wheel_radius}</wheel_radius>
+      <odom_publish_frequency>50</odom_publish_frequency>
+      <topic>/cmd_vel</topic>
+      <odom_topic>/odom</odom_topic>
+      <frame_id>odom</frame_id>
+      <child_frame_id>base_link</child_frame_id>
+      <tf_topic>/tf</tf_topic>
+    </plugin>
+  </gazebo>
+  <!-- ── Gazebo: Joint state publisher ─────────────────────────────────────── -->
+  <!-- Only acted on by Gazebo; real hardware uses the standalone
+       joint_state_publisher node instead (see guardian.launch.py). -->
+  <gazebo>
+    <plugin filename="gz-sim-joint-state-publisher-system"
+            name="gz::sim::systems::JointStatePublisher">
+      <topic>/joint_states</topic>
+    </plugin>
+  </gazebo>
 </robot>
